Commit message: feat(hand): different shader looks a bit better

File: public/hand/dg5f/dg5f_left.urdf (robot description, URDF)
Before this commit: robot dg5f_left, 28 links, 27 joints
Joints:
- joint lj_dg_3_2: origin xyz=0.01765 0.0 0.0265 rpy=0.0 1 0.0 -> xyz=0.01765 0.0 0.0265 rpy=0.0 1.5708 0.0
- joint lj_dg_4_2: origin xyz=0.01765 0.0 0.0265 rpy=0.0 1.4 0.0 -> xyz=0.01765 0.0 0.0265 rpy=0.0 1.5708 0.0
- joint lj_dg_5_2: origin xyz=0.0 0.028 0.0381 rpy=0.0 1.3 0.0 -> xyz=0.0 0.028 0.0381 rpy=0.0 1.5708 0.0
- joint lj_dg_5_4: origin xyz=0.0 0.0 0.0388 rpy=0.0 0.0 0.0 -> xyz=0.0 0.0 0.0388 rpy=0.0 1.0 0.0
