Commit message: feat: single-page pixel screens homepage
Replace the card grid and subpages with one page of full-screen
"screens" (About, Robotic Hands, Rocket Nozzle, Examsearch):

- dithered low-res backgrounds that crossfade between screens;
  arrows, keys, wheel, swipe and a slot indicator to navigate
- Read fades the background to the same picture at full res (live
  URDF hand aligned to its render, crisp characteristics chart,
  greyscale photo) with the write-up scrolling over it; the nozzle
  write-up has the 3D wireframe inline
- full-res assets and three.js prefetch when a screen is landed on
- responsive: render screens fit width on portrait phones
- scripts/make-art.sh regenerates screen images from gitignored
  source photos so only reduced images are published

Remove the nozzle/hand/examsearch subpages, unused collision and
hidden hand meshes, Tailwind leftovers and other dead assets.

Co-Authored-By: Claude Opus 5.5 <noreply@anthropic.com>

File: public/hand/dg5f/dg5f_left.urdf (robot description, URDF)
Before this commit: robot dg5f_left, 28 links, 27 joints
Links:
- link ll_dg_1_1: geometry visual mesh filename=package://meshes/dg5f_left/ll_dg_1_1.dae
- link ll_dg_1_2: geometry visual mesh filename=package://meshes/dg5f_left/ll_dg_1_2.dae
- link ll_dg_1_3: geometry visual mesh filename=package://meshes/dg5f_left/ll_dg_1_3.dae
- link ll_dg_1_4: geometry visual mesh filename=package://meshes/dg5f_left/ll_dg_1_4.dae
- link ll_dg_1_tip: geometry visual mesh filename=package://meshes/dg5f_left/ll_dg_1_tip.dae
- link ll_dg_2_1: geometry visual mesh filename=package://meshes/dg5f_left/ll_dg_2_1.dae
- link ll_dg_2_2: geometry visual mesh filename=package://meshes/dg5f_left/ll_dg_2_2.dae
- link ll_dg_2_3: geometry visual mesh filename=package://meshes/dg5f_left/ll_dg_2_3.dae
- link ll_dg_2_4: geometry visual mesh filename=package://meshes/dg5f_left/ll_dg_2_4.dae
- link ll_dg_2_tip: geometry visual mesh filename=package://meshes/dg5f_left/ll_dg_2_tip.dae
- link ll_dg_3_1: geometry visual mesh filename=package://meshes/dg5f_left/ll_dg_3_1.dae
- link ll_dg_3_2: geometry visual mesh filename=package://meshes/dg5f_left/ll_dg_3_2.dae
- link ll_dg_3_3: geometry visual mesh filename=package://meshes/dg5f_left/ll_dg_3_3.dae
- link ll_dg_3_4: geometry visual mesh filename=package://meshes/dg5f_left/ll_dg_3_4.dae
- link ll_dg_3_tip: geometry visual mesh filename=package://meshes/dg5f_left/ll_dg_3_tip.dae
- link ll_dg_4_1: geometry visual mesh filename=package://meshes/dg5f_left/ll_dg_4_1.dae
- link ll_dg_4_2: geometry visual mesh filename=package://meshes/dg5f_left/ll_dg_4_2.dae
- link ll_dg_4_3: geometry visual mesh filename=package://meshes/dg5f_left/ll_dg_4_3.dae
- link ll_dg_4_4: geometry visual mesh filename=package://meshes/dg5f_left/ll_dg_4_4.dae
- link ll_dg_4_tip: geometry visual mesh filename=package://meshes/dg5f_left/ll_dg_4_tip.dae
- link ll_dg_5_1: geometry visual mesh filename=package://meshes/dg5f_left/ll_dg_5_1.dae
- link ll_dg_5_2: geometry visual mesh filename=package://meshes/dg5f_left/ll_dg_5_2.dae
- link ll_dg_5_3: geometry visual mesh filename=package://meshes/dg5f_left/ll_dg_5_3.dae
- link ll_dg_5_4: geometry visual mesh filename=package://meshes/dg5f_left/ll_dg_5_4.dae
- link ll_dg_5_tip: geometry visual mesh filename=package://meshes/dg5f_left/ll_dg_5_tip.dae
- link ll_dg_base: geometry 
- link ll_dg_mount: geometry 
- link ll_dg_palm: geometry visual mesh filename=package://meshes/dg5f_left/ll_dg_palm.dae
